File: PCB_BatteryModule.sch (KiCad schematic (older format))
At the start: 71 parts, among them J1 Interconnect A, J2 Interconnect B, J3 Debug, J4 Button/Status, J5 Barrel_Jack, Q1 IRF7406, Q2 IRF7303, Q3 IRF7303, Q4 IRF7309, SW1 SW_Push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

Commit message: Add a pull-down resistor to the charger n-channel mosfet
Adding a pull-down resistor to the gate of the n-channel mosfet
prevents current from flowing through it when there is no charger voltage.
Parts:
- added R18: 380K, PCB_BatteryModule:C_0805_HandSoldering, symbol Device:R
Connections:
- net -BATT: now also R18.2
- net at Q4.2 (G), U7.13 (NDRV): now also R18.1
Changed lines of the file:
@@
 $EndComp
 Wire Wire Line
-	14350 7550 14150 7550
-Wire Wire Line
-	14650 7850 14150 7850
+	14350 7550 14300 7550
+Wire Wire Line
+	14650 7850 14300 7850
 Wire Wire Line
 	14650 7750 14650 7850
@@
 	1    0    0    1
 $EndComp
+$Comp
+L Device:R R18
+U 1 1 65B41F59
+P 14300 7700
+F 0 "R18" H 14370 7746 50  0000 L CNN
+F 1 "380K" H 14370 7655 50  0000 L CNN
+F 2 "PCB_BatteryModule:C_0805_HandSoldering" V 14230 7700 50  0001 C CNN
+F 3 "~" H 14300 7700 50  0001 C CNN
+	1    14300 7700
+	1    0    0    -1
+$EndComp
+Connection ~ 14300 7550
+Wire Wire Line
+	14300 7550 14150 7550
+Connection ~ 14300 7850
+Wire Wire Line
+	14300 7850 14150 7850
 $EndSCHEMATC

Commit message: Use the correct footprint for the button
Parts:
- SW1: footprint Button_Switch_SMD:SW_SPST_Omron_B3FS-100xP -> PCB_BatteryModule:CK_Switch_KSC_Series
Changed lines of the file:
@@
 F 0 "SW1" H 10700 2235 50  0000 C CNN
 F 1 "SW_Push" H 10700 2144 50  0000 C CNN
-F 2 "Button_Switch_SMD:SW_SPST_Omron_B3FS-100xP" H 10700 2150 50  0001 C CNN
+F 2 "PCB_BatteryModule:CK_Switch_KSC_Series" H 10700 2150 50  0001 C CNN
 F 3 "~" H 10700 2150 50  0001 C CNN
 	1    10700 1950

Commit message: Change the D1 footprint to be regular SMC one instead of the handsoldering version
Parts:
- D1: footprint Diodes_SMD:D_SMC_Handsoldering -> Diode_SMD:D_SMC
Changed lines of the file:
@@
 F 0 "D1" V 3254 9668 50  0000 L CNN
 F 1 "420mV 4A" V 3345 9668 50  0000 L CNN
-F 2 "Diodes_SMD:D_SMC_Handsoldering" V 3300 9600 50  0001 C CNN
+F 2 "Diode_SMD:D_SMC" V 3300 9600 50  0001 C CNN
 F 3 "~" V 3300 9600 50  0001 C CNN
 	1    3300 9600
